File: keyboard/keyboard.kicad_pcb (KiCad board)
At the start: 2 copper layers, 323.9 x 109.5 mm, 145 parts, among them J1 col, J10 col, J11 col, J12 col, J13 col, J14 col, J15 row, J16 row, J17 row, J18 row, J19 row, J2 col, J3 col, J4 col, J5 col, J6 col, J7 col, J8 col, J9 col

Commit message: Updated with reference switches
Parts:
- S1, S10, S11, S12, S13, S16, S17, S18, S19, S2, S20, S21, S22, S23, S24, S25, S26, S27, S3, S30, S31, S32, S33, S34, S35, S36, S37, S38, S39, S4, S40, S43, S44, S45, S46, S47, S48, S49, S5, S50, S51, S52, S55, S59, S6, S60, S61, S62, S63, S7, S8, S9: footprint Button_Switch_Keyboard:SW_Cherry_MX_1.00u_PCB -> sandpiperfootprints:SW_Cherry_MX_1.00u_PCB
Connections:
- D1 pad 2: Net-(D1-A) -> unconnected-(D1-A-Pad2)
- S1 pad 2: Net-(D1-A) -> unconnected-(S1-Pad2)
Routing:
- net Net-(D1-A): track 6.59 -> 0.00 mm
- net (no net): track 0.00 -> 6.59 mm
