File: keyboard/keyboard.kicad_pcb (KiCad board)
At the start: 2 copper layers, 323.9 x 109.5 mm, 145 parts, among them J1 col, J10 col, J11 col, J12 col, J13 col, J14 col, J15 row, J16 row, J17 row, J18 row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

Commit message: USB keyboard instead
Parts:
- removed J10, J11, J12, J13, J14, J4, J5, J6, J7, J8, J9: col, TestPoint:TestPoint_THTPad_2.0x2.0mm_Drill1.0mm
- removed J15, J16, J17, J18, J19: row, TestPoint:TestPoint_THTPad_2.0x2.0mm_Drill1.0mm
- added C1: 1uF, Capacitor_SMD:C_0805_2012Metric, B.Cu at (339.1, 46.3)
- added C2: 0.1uF, Capacitor_SMD:C_0805_2012Metric, B.Cu at (335.1, 58.2)
- added C3: 0.1uF, Capacitor_SMD:C_0805_2012Metric, B.Cu at (318.7, 47.5)
- added C4: 0.1uF, Capacitor_SMD:C_0805_2012Metric, B.Cu at (323.1, 35.0)
- added C5: 10uF, Capacitor_SMD:C_0805_2012Metric, B.Cu at (333.1, 35.0)
- added C6: 22pF, Capacitor_SMD:C_0805_2012Metric, B.Cu at (328.6, 58.2)
- added C7: 22pF, Capacitor_SMD:C_0805_2012Metric, B.Cu at (322.3, 53.9)
- added R1: 10K, Resistor_SMD:R_0805_2012Metric, B.Cu at (318.9, 38.6)
- added R2: 22K, Resistor_SMD:R_0805_2012Metric, B.Cu at (339.1, 41.0)
- added R3: 22K, Resistor_SMD:R_0805_2012Metric, B.Cu at (339.1, 43.7)
- added R4: 10K, Resistor_SMD:R_0805_2012Metric, B.Cu at (334.1, 54.2)
- added REF**: MountingHole_2.2mm_M2, MountingHole:MountingHole_2.2mm_M2, F.Cu at (38.4, 117.3)
- added REF**: MountingHole_2.2mm_M2, MountingHole:MountingHole_2.2mm_M2, F.Cu at (345.9, 30.5)
- added REF**: MountingHole_2.2mm_M2, MountingHole:MountingHole_2.2mm_M2, F.Cu at (351.5, 122.0)
- added SW1: SW_Push, Button_Switch_SMD:SW_Tactile_SPST_NO_Straight_CK_PTS636Sx25SMTRLFS, B.Cu at (340.8, 53.3)
- added U1: ATmega32U4-A, Package_QFP:TQFP-44_10x10mm_P0.8mm, B.Cu at (328.1, 44.3)
- added Y1: 16MHz, Crystal:Crystal_SMD_3225-4Pin_3.2x2.5mm, B.Cu at (326.5, 54.8)
- J1: value col -> USB_C_Receptacle; footprint TestPoint:TestPoint_THTPad_2.0x2.0mm_Drill1.0mm -> Connector_USB:USB_C_Receptacle_GCT_USB4085
- J2: value col -> BANK_35; footprint TestPoint:TestPoint_THTPad_2.0x2.0mm_Drill1.0mm -> Connector_PinHeader_2.54mm:PinHeader_2x20_P2.54mm_Vertical
- J3: value col -> BANK_33; footprint TestPoint:TestPoint_THTPad_2.0x2.0mm_Drill1.0mm -> Connector_PinHeader_2.54mm:PinHeader_2x20_P2.54mm_Vertical
- S14: footprint Button_Switch_Keyboard:SW_Cherry_MX_2.00u_PCB -> sandpiperfootprints:SW_Cherry_MX_1.00u_PCB
- S15, S28: footprint Button_Switch_Keyboard:SW_Cherry_MX_1.50u_PCB -> sandpiperfootprints:SW_Cherry_MX_1.00u_PCB
- S29: footprint Button_Switch_Keyboard:SW_Cherry_MX_1.75u_PCB -> sandpiperfootprints:SW_Cherry_MX_1.00u_PCB
- S54: value LeftFunction -> LeftCtl
- S55: value LeftCtl -> Special
- moved J2 138.9 mm to (404.1, 49.6), turned to 0 degrees
- moved J1 102.0 mm to (343.5, 45.4), turned to 90 degrees
- moved J3 100.3 mm to (356.0, 49.6), turned to 0 degrees
Connections:
- D1 pad 2: unconnected-(D1-A-Pad2) -> Net-(D1-A)
- J2 pad 1: Column 1 -> unconnected-(J2-Pin_1-Pad1)
- J3 pad 1: Column 2 -> unconnected-(J3-Pin_1-Pad1)
- S1 pad 2: unconnected-(S1-Pad2) -> Net-(D1-A)
- S29 pad 1: Column 1 -> Column 0
- S30 pad 1: Column 2 -> Column 1
- S31 pad 1: Column 3 -> Column 2
- S32 pad 1: Column 4 -> Column 3
- S33 pad 1: Column 5 -> Column 4
- S34 pad 1: Column 6 -> Column 5
- S35 pad 1: Column 7 -> Column 6
- S36 pad 1: Column 8 -> Column 7
- S37 pad 1: Column 9 -> Column 8
- S38 pad 1: Column 10 -> Column 9
- S39 pad 1: Column 11 -> Column 10
- S40 pad 1: Column 12 -> Column 11
- S41 pad 1: Column 13 -> Column 12
- S60 pad 1: Column 13 -> Column 12
Routing:
- net Column 0: track 340.0 -> 475.5 mm, vias 0 -> 1
- net Column 2: track 313.5 -> 431.2 mm, vias 0 -> 1
- net Column 1: track 338.8 -> 454.6 mm, vias 0 -> 1
- net Column 6: track 249.8 -> 356.1 mm, vias 0 -> 1
- net Column 5: track 260.6 -> 364.8 mm, vias 0 -> 1
- net Column 3: track 287.1 -> 390.3 mm, vias 0 -> 1
- net Column 4: track 272.3 -> 374.6 mm, vias 0 -> 1
- net +5V: track 0.00 -> 72.4 mm
- net Row 0: track 354.1 -> 293.2 mm
- net Row 4: track 313.8 -> 367.1 mm
- net Row 1: track 339.7 -> 288.1 mm
- net Column 13: track 134.0 -> 108.4 mm, vias 0 -> 1
- net Row 2: track 324.3 -> 299.9 mm
- net Column 9: track 196.6 -> 209.1 mm, vias 0 -> 1
- net Column 12: track 145.8 -> 158.1 mm, vias 0 -> 1
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- added copper zone on B.Cu, net GND
- added copper zone on F.Cu, net GND
- removed copper zone on B.Cu, net (none)
- removed copper zone on F.Cu, net (none)
Other:
- board size 323.9 x 109.5 mm -> 378.5 x 106 mm
- board text added: "ETH"
- board text added: "HDMI"
- board text added: "Zynq7020"
- board text added: "sandpiper v0002 (c)2025 Engin Cilasun"
- board text removed: "sandpiper v0001 (c)2025 Engin Cilasun"

Commit message: updated pcb and enclosure
Parts:
- J2, J3: moved to B.Cu
- moved J2 2.54 mm to (406.6, 49.6), turned to 180 degrees
- moved J3 2.54 mm to (358.5, 49.6), turned to 180 degrees

Commit message: Updated keyboard with fixes, also much smaller
Parts:
- removed J2: BANK_35, Connector_PinHeader_2.54mm:PinHeader_2x20_P2.54mm_Vertical
- removed J3: BANK_33, Connector_PinHeader_2.54mm:PinHeader_2x20_P2.54mm_Vertical
- removed the REF** at (351.5, 122.0)
- added C8: 100nF, Capacitor_SMD:C_0805_2012Metric, B.Cu at (329.2, 35.0)
- added J4: ISP, Connector_PinHeader_2.54mm:PinHeader_2x03_P2.54mm_Vertical, B.Cu at (340.8, 60.4)
- SW1: value SW_Push -> RESET
- moved REF** 10.5 mm to (34.0, 127.0)
- moved REF** 1.34 mm to (345.5, 29.2)
Connections:
- net Net-(U1-~{RESET}) renamed RESET
- J1 pad A1: Net-(J1-GND-PadA1) -> GND
- J1 pad A12: Net-(J1-GND-PadA1) -> GND
- J1 pad B1: Net-(J1-GND-PadA1) -> GND
- J1 pad B12: Net-(J1-GND-PadA1) -> GND
- J1 pad S1: unconnected-(J1-SHIELD-PadS1) -> GND
- U1 pad 10: unconnected-(U1-PB2-Pad10) -> MOSI
- U1 pad 11: Column 0 -> MISO
- U1 pad 12: unconnected-(U1-PB7-Pad12) -> Column 0
- U1 pad 42: unconnected-(U1-AREF-Pad42) -> Net-(U1-AREF)
- U1 pad 8: unconnected-(U1-PB0-Pad8) -> CS
- U1 pad 9: unconnected-(U1-PB1-Pad9) -> SCK
Routing:
- net MOSI: track 0.00 -> 22.0 mm, vias 0 -> 1
- net SCK: track 0.00 -> 18.5 mm
- net MISO: track 0.00 -> 15.4 mm
- net RESET: track 7.49 -> 20.7 mm, vias 0 -> 1
- net +5V: track 72.4 -> 82.3 mm
- net Net-(U1-AREF): track 0.00 -> 3.79 mm
- net Net-(J1-GND-PadA1): track 2.70 -> 0.00 mm
- net Row 3: track 317.6 -> 318.2 mm
- net GND: vias 2 -> 7
Other:
- board size 378.5 x 106 mm -> 319.5 x 106 mm
- board text added: "ATmega32U4-A"
- board text added: "AVRISP"
- board text added: "RESET"
- board text added: "sandpiper v0003 (c)2025 Engin Cilasun"
- board text removed: "sandpiper v0002 (c)2025 Engin Cilasun"
